File: input switch /input switch .kicad_sch (KiCad schematic)
At the start: 11 parts, among them IC1 MCP23008T-E_SS, IC2 TLP293-4_GB,E, IC3 TLP293-4_GB,E, J1 BHR-06-VUA

Commit message: likely all done with v1, mainboard obsolete
Parts:
- gave numbers to parts that had none: 2
