File: psu/psu.kicad_sch (KiCad schematic)
At the start: 6 parts, among them J1 26-60-4023, J2 26-60-4023

Commit message: likely all done with v1, mainboard obsolete
Parts:
- removed J2: 26-60-4023, Samacsys:26604023, symbol Samacsys:26-60-4023
- added H1, H2, H3, H4: MountingHole, MountingHole:MountingHole_3.2mm_M3_ISO7380, symbol Mechanical:MountingHole
- added J2: 4628, Samacsys:4628, symbol Samacsys:4628
- added J3: BHR-06-VUA, Samacsys:SHDR6W64P254_2X3_1522X880X920P, symbol Samacsys:BHR-06-VUA
Connections:
- net +5V: now also J3.1, J3.3, J3.5
- net GNDD: now also J3.2, J3.4, J3.6
- net at J1.1: now also J2.1; no longer PS1.5 (AC_IN_(N))
- new net: J2.2, PS1.5 (AC_IN_(N))
- no-connect marks 0 -> 1
Other:
- moved on the sheet: J1
