File: Volume front panel/Volume front panel.kicad_pcb (KiCad board)
At the start: 2 copper layers, 199 x 31.9 mm, 33 parts, among them IC1 TLC5947DAPR, J1 BHR-06-VUA, J2 BHR-06-VUA, U1 PEC11R-4330F-S0012, U2 PEC11R-4330F-S0012, U3 TSOP39238

Commit message: almost made 2040 raw
Parts:
- removed A1: Arduino_Nano_v3.x, Module:Arduino_Nano
- removed the C1 at (248.0, 108.0)
- removed the C4 at (209.1, 110.4)
- removed J2: BHR-06-VUA, Samacsys:SHDR6W64P254_2X3_1522X880X920P
- removed the R9 at (106.0, 96.7)
- added C2: 15p, Capacitor_SMD:C_1206_3216Metric, F.Cu at (101.0, 106.0)
- added C5: 10uf, Capacitor_SMD:C_1206_3216Metric, F.Cu at (129.0, 98.8)
- added C8: 15p, Capacitor_SMD:C_1206_3216Metric, F.Cu at (109.5, 105.8)
- added IC1: W25Q16JVUXIQ_TR, Samacsys:SON50P300X200X60-9N, F.Cu at (125.5, 95.2)
- added IC2: TS02-66-80-BK-160-LCR-D, Samacsys:TS026680BK160LCRD, F.Cu at (81.8, 91.2)
- added R1: 5.1k, Resistor_SMD:R_1206_3216Metric, F.Cu at (97.5, 100.2)
- added R15: 27.4, Resistor_SMD:R_1206_3216Metric, F.Cu at (122.0, 101.5)
- added R16: 27.4, Resistor_SMD:R_1206_3216Metric, F.Cu at (121.8, 104.0)
- added R2: 5.1k, Resistor_SMD:R_1206_3216Metric, F.Cu at (94.5, 100.2)
- added R3: 1k, Resistor_SMD:R_1206_3216Metric, F.Cu at (124.8, 90.8)
- added R4: 10k, Resistor_SMD:R_1206_3216Metric, F.Cu at (128.0, 95.2)
- added U4: MIC5205-3.3YM5, Package_TO_SOT_SMD:SOT-23-5, F.Cu at (131.8, 88.8)
- added U5: RP2040, Package_DFN_QFN:QFN-56-1EP_7x7mm_P0.4mm_EP3.2x3.2mm, F.Cu at (115.0, 97.2)
- added Y1: ABM8-12.000MHZ-B2-T, Samacsys:ABM810000MHZ12D2W, F.Cu at (105.5, 106.0)
- J1: value BHR-06-VUA -> 10159872-00011LF; footprint Samacsys:SHDR6W64P254_2X3_1522X880X920P -> Samacsys:1015987200011LF
- R11: value 4.7k -> 1k
- moved J1 152.4 mm to (96.8, 91.5), turned to 180 degrees
- moved C11 12.2 mm to (142.8, 112.3)
- moved R14 2.05 mm to (140.2, 112.3)
- moved R11 1.68 mm to (105.2, 101.5), turned to 180 degrees
- moved C12 1.46 mm to (140.8, 95.8)
- moved R17 1.46 mm to (140.7, 100.7)
- moved R18 1.46 mm to (140.8, 98.2)
- renumbered C2 to C1, C9 to C10, C10 to C11, C11 to C12, C12 to C13, C5 to C4, C8 to C9, IC1 to IC3, R6 to R10, R7 to R12, R8 to R13, R10 to R14, R12 to R17, R13 to R18, R1 to R5, R2 to R6, R3 to R7, R4 to R8, R5 to R9
Connections:
- net Net-(A1-D2) renamed enc2a
- net Net-(A1-D3) renamed enc1a
- net Net-(A1-D4) renamed enc1b
- net Net-(A1-D5) renamed enc2b
- net Net-(A1-D6) renamed enc1press
- net Net-(A1-D7) renamed enc2press
- J1 pad 1: +5V -> unconnected-(J1-MH1-Pad1)
- J1 pad 2: GNDD -> unconnected-(J1-MH2-Pad2)
- J1 pad 3: +5V -> unconnected-(J1-MH3-Pad3)
- J1 pad 4: GNDD -> unconnected-(J1-MH4-Pad4)
- R10 pad 2: +5V -> +3.3V
- R11 pad 1: SCL -> Net-(Y1-X2)
- R11 pad 2: +5V -> XIN
- R12 pad 1: +5V -> +3.3V
- R14 pad 1: +5V -> +3.3V
- R6 pad 2: +5V -> +3.3V
- R7 pad 1: +5V -> +3.3V
Routing:
- net +5V: track 294.6 -> 27.1 mm
- net SCL: track 126.4 -> 0.00 mm, vias 1 -> 0
- net enc1press: track 135.3 -> 9.36 mm, vias 1 -> 0
- net enc1a: track 144.4 -> 23.5 mm
- net SDA: track 119.3 -> 0.00 mm, vias 1 -> 0
- net enc1b: track 152.2 -> 33.0 mm, vias 1 -> 0
- net +3.3V: track 0.00 -> 82.0 mm
- net blank: track 54.5 -> 0.00 mm, vias 2 -> 0
- net xlat: track 54.1 -> 0.00 mm
- net sclk: track 47.7 -> 0.00 mm, vias 2 -> 0
- net IR: track 52.7 -> 8.29 mm, vias 4 -> 0
- net data: track 43.3 -> 0.00 mm
- net (no net): track 0.00 -> 24.2 mm
- net enc2b: track 35.7 -> 15.2 mm, vias 1 -> 0
- net enc2press: track 40.7 -> 25.2 mm
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
Commit message: pico front panel so easy
Parts:
- removed the C2 at (101.0, 106.0)
- removed the C5 at (129.0, 98.8)
- removed the C8 at (109.5, 105.8)
- removed the IC1 at (125.5, 95.2)
- removed IC2: TS02-66-80-BK-160-LCR-D, Samacsys:TS026680BK160LCRD
- removed the R1 at (97.5, 100.2)
- removed the R11 at (105.2, 101.5)
- removed R15, R16: 27.4, Resistor_SMD:R_1206_3216Metric
- removed the R2 at (94.5, 100.2)
- removed the R3 at (124.8, 90.8)
- removed the R4 at (128.0, 95.2)
- removed U5: RP2040, Package_DFN_QFN:QFN-56-1EP_7x7mm_P0.4mm_EP3.2x3.2mm
- removed Y1: ABM8-12.000MHZ-B2-T, Samacsys:ABM810000MHZ12D2W
- added J2: 26-60-4023, Samacsys:26604023, F.Cu at (212.3, 98.9)
- added PS1: TMPW_5-105, Samacsys:TMPW5112, F.Cu at (174.6, 89.0)
- J1: value 10159872-00011LF -> TFM-105-01-F-D; footprint Samacsys:1015987200011LF -> Samacsys:TFM-105-XX-YYY-D
- U4: value MIC5205-3.3YM5 -> Pico; footprint Package_TO_SOT_SMD:SOT-23-5 -> MCU_RaspberryPi_and_Boards:RPi_Pico_SMD_TH
- moved J1 29.4 mm to (67.5, 88.5), turned to 0 degrees
- moved U4 26.5 mm to (108.2, 101.0), turned to 90 degrees
- moved C2 5.25 mm to (70.0, 95.2)
- moved C6 1.46 mm to (224.0, 105.5)
- moved R8 1.08 mm to (224.0, 108.0)
- renumbered C13 to C10, C3 to C2, C4 to C3, C6 to C4, C7 to C5, C9 to C6, C10 to C7, C11 to C8, C12 to C9, IC3 to IC1, R5 to R1, R17 to R10, R18 to R11, R6 to R2, R7 to R3, R8 to R4, R9 to R5, R10 to R6, R12 to R7, R13 to R8, R14 to R9
Connections:
- J1 pad 1: unconnected-(J1-MH1-Pad1) -> +5V
- J1 pad 2: unconnected-(J1-MH2-Pad2) -> +5V
- J1 pad 3: unconnected-(J1-MH3-Pad3) -> GNDD
- J1 pad 4: unconnected-(J1-MH4-Pad4) -> +5V
- U4 pad 1: +5V -> enc1a
- U4 pad 2: GNDD -> enc1b
- U4 pad 3: +5V -> GNDD
- U4 pad 4: GNDD -> enc1press
- U4 pad 5: +3.3V -> unconnected-(U4-GPIO3-Pad5)
Routing:
- net +3.3V: track 82.0 -> 248.2 mm, vias 0 -> 7
- net +5V: track 27.1 -> 172.8 mm, vias 0 -> 2
- net enc2press: track 25.2 -> 128.7 mm
- net enc2b: track 15.2 -> 101.6 mm
- net enc2a: track 43.2 -> 127.4 mm
- net SER1: track 0.00 -> 45.3 mm
- net xlat: track 0.00 -> 44.2 mm
- net SRCLK1: track 0.00 -> 41.8 mm
- net blank: track 0.00 -> 39.9 mm, vias 0 -> 2
- net RCLK1: track 0.00 -> 37.6 mm
- net data: track 0.00 -> 35.4 mm
- net sclk: track 0.00 -> 31.8 mm
- net enc1press: track 9.36 -> 37.2 mm
- net (no net): track 24.2 -> 0.00 mm
- net Net-(PS1-AC_IN_(N)): track 0.00 -> 20.7 mm
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Other:
- board size 199 x 31.9 mm -> 186.5 x 31.9 mm
