File: Volume front panel/Volume front panel.kicad_pcb (KiCad board)
At the start: 2 copper layers, 186.5 x 31.9 mm, 30 parts, among them IC1 TLC5947DAPR, J1 TFM-105-01-F-D, J2 26-60-4023, U1 PEC11R-4330F-S0012, U2 PEC11R-4330F-S0012, U3 TSOP39238, U4 Pico

Commit message: little neatening
Routing:
- net +3.3V: track 248.2 -> 250.8 mm
- net enc2press: track 128.7 -> 129.2 mm

Commit message: moved control to side, added electrolytic caps
Parts:
- added C11: VZL221M1CTR-0607, Samacsys:CAPAE660X800N, F.Cu at (215.8, 89.2)
- added C12: VZL221M1CTR-0607, Samacsys:CAPAE660X800N, F.Cu at (207.0, 89.2)
- added L1: 150uh, Inductor_SMD:L_Coilcraft_XAL6060-XXX, F.Cu at (207.2, 97.8)
- moved J2 6.22 mm to (209.6, 104.5), turned to 90 degrees
- moved PS1 5.77 mm to (168.8, 88.5)
Connections:
- PS1 pad 2: +5V -> Net-(PS1-+VOUT)
Routing:
- net Net-(PS1-+VOUT): track 0.00 -> 47.4 mm
- net +5V: track 172.8 -> 189.3 mm
- net Net-(PS1-AC_IN_(L)): track 19.2 -> 12.2 mm
- net +3.3V: track 250.8 -> 252.2 mm, vias 7 -> 9
- net Net-(PS1-AC_IN_(N)): track 20.7 -> 21.3 mm
- net GNDD: vias 23 -> 25
