File: Audioboard/Audioboard.kicad_pcb (KiCad board)
At the start: 2 copper layers, 51 x 58 mm, 48 parts, among them J1 10129381-908001BLF, J2 10129381-908001BLF, K1 RELAY_G6K, K2 RELAY_G6K, K3 RELAY_G6K, K4 RELAY_G6K, K5 RELAY_G6K, K6 RELAY_G6K, P1 audioIn, P2 audioOut

Commit message: likely all done with v1, mainboard obsolete
Parts:
- removed D1, D2, D3, D4, D5, D6: 1N4001, Diode_SMD:D_SMA
- removed P1: audioIn, RlxPassiveFootprints:PIN_ARRAY_4x1
- removed P2: audioOut, RlxPassiveFootprints:PIN_ARRAY_4x1
- added C1: .1uf, Capacitor_SMD:C_1206_3216Metric, F.Cu at (86.4, 64.2)
- added C2: UUD1V101MNL1GS, Samacsys:CAPAE830X1050N, F.Cu at (99.0, 70.2)
- added C3: .1uf, Capacitor_SMD:C_1206_3216Metric, F.Cu at (85.0, 50.8)
- added C4: .1uf, Capacitor_SMD:C_1206_3216Metric, F.Cu at (95.0, 50.8)
- added C5: .1uf, Capacitor_SMD:C_1206_3216Metric, F.Cu at (85.0, 45.5)
- added C6: .1uf, Capacitor_SMD:C_1206_3216Metric, F.Cu at (95.0, 45.2)
- added C7: 10uf, Capacitor_SMD:C_1206_3216Metric, F.Cu at (86.0, 42.0)
- added C8: 1uf, Capacitor_SMD:C_1206_3216Metric, F.Cu at (86.0, 37.0)
- added IC1: ULN2003ADR, Samacsys:SOIC127P600X175-16N, F.Cu at (83.5, 57.6)
- added IC2: MCP23017T-E_SS, Samacsys:SOP65P780X200-28N, F.Cu at (93.6, 58.5)
- added IC3: ISO7740FDBQR, Samacsys:SOP64P600X175-16N, F.Cu at (100.0, 48.0)
- added IC4: ISO7740FDBQR, Samacsys:SOP64P600X175-16N, F.Cu at (90.0, 48.0)
- added IC5: ULN2003ADR, Samacsys:SOIC127P600X175-16N, F.Cu at (95.0, 39.0)
- added IC6: ZXTR2105FQ-7, Samacsys:SOT96P240X110-3N, F.Cu at (83.0, 39.0)
- added J3: BHR-06-VUA, Samacsys:SHDR6W64P254_2X3_1522X880X920P, F.Cu at (84.0, 80.6)
- added J4: 61201021621, Samacsys:SHDR10W64P254_2X5_2036X885X925P, F.Cu at (91.5, 29.2)
- added JPVCC1: VCC, Jumper:SolderJumper-3_P1.3mm_Open_Pad1.0x1.5mm, F.Cu at (100.8, 61.5)
- added R1: 4.7k, Resistor_SMD:R_1206_3216Metric, F.Cu at (102.2, 57.5)
- added R12: 4.7k, Resistor_SMD:R_1206_3216Metric, F.Cu at (99.8, 57.5)
- J1, J2: value 10129381-908001BLF -> BHR-06-VUA; footprint Samacsys:10129381908001BLF -> Samacsys:SHDR6W64P254_2X3_1522X880X920P
- moved J2 46.6 mm to (38.4, 52.5), turned to -90 degrees
- moved H2 20.0 mm to (100.0, 30.0)
- moved H4 20.0 mm to (100.0, 80.0)
- moved J1 19.8 mm to (84.0, 71.1), turned to 0 degrees
- renumbered R9 to R10, R10 to R11, R11 to R13, R12 to R14, R13 to R15, R14 to R16, R15 to R17, R16 to R18, R17 to R19, R1 to R2, R18 to R20, R19 to R21, R20 to R22, R21 to R23, R22 to R24, R23 to R25, R24 to R26, R25 to R27, R26 to R28, R27 to R29, R2 to R3, R28 to R30, R3 to R4, R4 to R5, R5 to R6, R6 to R7, R7 to R8, R8 to R9
Connections:
- J1 pad 3: r3 -> GNDD
- J1 pad 4: r2 -> GNDD
- J1 pad 5: r1 -> SCL
- J1 pad 6: r0 -> SDA
- J2 pad 1: +5V -> outR
- J2 pad 2: +5V -> outL
- J2 pad 3: r3 -> AGND
- J2 pad 4: r2 -> AGND
- J2 pad 5: r1 -> inR
- J2 pad 6: r0 -> inL
- K1 pad 4: Net-(P1-P1) -> inL
- K1 pad 5: Net-(P1-P4) -> inR
- K6 pad 3: Net-(P2-P1) -> outL
- K6 pad 6: Net-(P2-P4) -> outR
- R2 pad 2: Net-(P1-P4) -> inR
- R25 pad 1: Net-(P2-P4) -> outR
- R26 pad 1: Net-(P2-P1) -> outL
- R29 pad 1: Net-(P2-P4) -> outR
- R3 pad 2: Net-(P1-P1) -> inL
- R30 pad 1: Net-(P2-P1) -> outL
Routing:
- net +5V: track 106.6 -> 210.9 mm, vias 6 -> 16
- net outR: track 0.00 -> 38.0 mm
- net VCC: track 0.00 -> 33.9 mm, vias 0 -> 1
- net r2: track 48.7 -> 16.6 mm
- net +5VI: track 0.00 -> 30.1 mm, vias 0 -> 4
- net Net-(IC5-7C): track 0.00 -> 27.6 mm
- net Net-(IC5-6C): track 0.00 -> 25.4 mm
- net Net-(P2-P1): track 23.6 -> 0.00 mm
- net SCL: track 0.00 -> 23.5 mm
- net Net-(P2-P4): track 23.4 -> 0.00 mm
- net Net-(IC5-5C): track 0.00 -> 21.8 mm
- net inR: track 0.00 -> 21.5 mm
- net r0: track 56.0 -> 34.5 mm, vias 1 -> 2
- net outL: track 0.00 -> 21.1 mm
- net r1: track 46.1 -> 26.2 mm, vias 1 -> 2
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- added copper zone on B.Cu, net GNDA
- added copper zone on F.Cu, net GNDA
- added copper zone on B.Cu, net GNDD
- added copper zone on F.Cu, net GNDD
Other:
- board size 51 x 58 mm -> 70 x 58 mm

Commit message: somehow maybe done
Parts:
- removed C3, C4, C5, C6: .1uf, Capacitor_SMD:C_1206_3216Metric
- removed C7: 10uf, Capacitor_SMD:C_1206_3216Metric
- removed C8: 1uf, Capacitor_SMD:C_1206_3216Metric
- removed IC2: MCP23017T-E_SS, Samacsys:SOP65P780X200-28N
- removed IC3, IC4: ISO7740FDBQR, Samacsys:SOP64P600X175-16N
- removed IC5: ULN2003ADR, Samacsys:SOIC127P600X175-16N
- removed IC6: ZXTR2105FQ-7, Samacsys:SOT96P240X110-3N
- removed J2: BHR-06-VUA, Samacsys:SHDR6W64P254_2X3_1522X880X920P
- removed the J4 at (91.5, 29.2)
- removed JPVCC1: VCC, Jumper:SolderJumper-3_P1.3mm_Open_Pad1.0x1.5mm
- removed the R1 at (102.2, 57.5)
- added J3: TFM-105-01-F-D, Samacsys:TFM-105-XX-YYY-D, F.Cu at (18.0, 53.5)
- added K1: RELAY_G6K, RlxPassiveFootprints:G6K-2F-Y, F.Cu at (187.0, 83.0)
- added K2: RELAY_G6K, RlxPassiveFootprints:G6K-2F-Y, F.Cu at (187.0, 98.5)
- added K3: RELAY_G6K, RlxPassiveFootprints:G6K-2F-Y, F.Cu at (187.0, 113.5)
- added K4: RELAY_G6K, RlxPassiveFootprints:G6K-2F-Y, F.Cu at (187.0, 127.5)
- J1: value BHR-06-VUA -> PJRAS4X2U01AUX; footprint Samacsys:SHDR6W64P254_2X3_1522X880X920P -> Samacsys:PJRAS4X2U01AUX
- moved R1 193.6 mm to (230.4, 136.7), turned to 180 degrees
- moved R26 189.0 mm to (230.5, 73.4), turned to 180 degrees
- moved R3 188.6 mm to (230.4, 132.7), turned to 180 degrees
- moved R28 186.0 mm to (230.5, 77.4), turned to 0 degrees
- moved R5 183.6 mm to (230.4, 128.7), turned to 180 degrees
- moved R2 183.4 mm to (212.4, 136.7), turned to 0 degrees
- moved R24 183.1 mm to (230.5, 81.4), turned to 180 degrees
- moved K5 183.0 mm to (221.4, 132.7), turned to -90 degrees
- moved R22 180.4 mm to (230.5, 85.4), turned to 180 degrees
- moved R7 178.7 mm to (230.4, 124.7), turned to 0 degrees
- moved R4 178.1 mm to (212.4, 132.7), turned to 0 degrees
- moved R20 175.4 mm to (230.5, 93.4), turned to 180 degrees
- moved K10 175.2 mm to (221.5, 77.4), turned to -90 degrees
- moved R9 173.8 mm to (230.4, 120.7), turned to 180 degrees
- moved R18 173.1 mm to (230.5, 97.4), turned to 180 degrees
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- renumbered J3 to J4, K6 to K10, K1 to K5, K2 to K6, K3 to K7, K4 to K8, K5 to K9, R2 to R1, R11 to R10, R12 to R11, R13 to R12, R14 to R13, R15 to R14, R16 to R15, R17 to R16, R18 to R17, R19 to R18, R20 to R19, R3 to R2, R21 to R20, R22 to R21, R23 to R22, R24 to R23, R25 to R24, R26 to R25, R27 to R26, R28 to R27, R29 to R28, R30 to R29, R4 to R3, R5 to R4, R6 to R5, R7 to R6, R8 to R7, R9 to R8, R10 to R9
Connections:
- IC1 pad 1: Net-(IC1-1B) -> unconnected-(IC1-1B-Pad1)
- IC1 pad 2: Net-(IC1-2B) -> unconnected-(IC1-2B-Pad2)
- IC1 pad 3: Net-(IC1-3B) -> unconnected-(IC1-3B-Pad3)
- IC1 pad 4: Net-(IC1-4B) -> unconnected-(IC1-4B-Pad4)
- IC1 pad 5: Net-(IC1-5B) -> unconnected-(IC1-5B-Pad5)
- IC1 pad 6: Net-(IC1-6B) -> unconnected-(IC1-6B-Pad6)
- R11 pad 1: Net-(IC2-~{RESET}) -> unconnected-(R11-Pad1)
Routing:
- net (no net): track 0.00 -> 319.8 mm, vias 0 -> 21
- net VCC: track 33.9 -> 0.00 mm, vias 1 -> 0
- net +5VI: track 30.1 -> 0.00 mm, vias 4 -> 0
- net Net-(IC5-7C): track 27.6 -> 0.00 mm
- net Net-(IC5-6C): track 25.4 -> 0.00 mm
- net Net-(IC5-5C): track 21.8 -> 0.00 mm
- net Net-(IC5-4C): track 17.7 -> 0.00 mm
- net GNDA: track 15.9 -> 0.00 mm, vias 12 -> 0
- net Net-(IC5-3C): track 13.7 -> 0.00 mm, vias 2 -> 0
- net Net-(IC2-GPA0): track 12.6 -> 0.00 mm
- net Net-(IC2-GPA1): track 11.7 -> 0.00 mm
- net Net-(IC2-GPA2): track 10.7 -> 0.00 mm
- net Net-(IC5-2C): track 10.6 -> 0.00 mm, vias 2 -> 0
- net Net-(IC2-GPA3): track 9.79 -> 0.00 mm
- net Net-(IC2-GPA5): track 9.68 -> 0.00 mm
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- added copper zone on B.Cu, net (none)
- added copper zone on F.Cu, net (none)
- removed copper zone on B.Cu, net GNDA
- removed copper zone on F.Cu, net GNDA
