File: Audioboard/audio-attenuator.kicad_sch (KiCad schematic)
At the start: 48 parts, among them J1 10129381-908001BLF, J2 10129381-908001BLF, K1 RELAY_G6K, K2 RELAY_G6K, K3 RELAY_G6K, K4 RELAY_G6K, K5 RELAY_G6K, K6 RELAY_G6K, P1 audioIn, P2 audioOut

Commit message: likely all done with v1, mainboard obsolete
Parts:
- removed D1, D2, D3, D4, D5, D6: 1N4001, Diode_SMD:D_SMA, symbol Device:D
- removed J1, J2: 10129381-908001BLF, Samacsys:10129381908001BLF, symbol Samacsys:10129381-908001BLF
- removed P1: audioIn, RlxPassiveFootprints:PIN_ARRAY_4x1, symbol relaixedPassive-rescue:CONN_4
- removed P2: audioOut, RlxPassiveFootprints:PIN_ARRAY_4x1, symbol relaixedPassive-rescue:CONN_4
- added C1, C3, C4, C5, C6: .1uf, Capacitor_SMD:C_1206_3216Metric, symbol Device:C_Small
- added C2: UUD1V101MNL1GS, Samacsys:CAPAE830X1050N, symbol Samacsys:UUD1V101MNL1GS
- added C7: 10uf, Capacitor_SMD:C_1206_3216Metric, symbol Device:C_Small
- added C8: 1uf, Capacitor_SMD:C_1206_3216Metric, symbol Device:C_Small
- added IC1, IC5: ULN2003ADR, Samacsys:SOIC127P600X175-16N, symbol Samacsys:ULN2003ADR
- added IC2: MCP23017T-E_SS, Samacsys:SOP65P780X200-28N, symbol Samacsys:MCP23017T-E_SS
- added IC3, IC4: ISO7740FDBQR, Samacsys:SOP64P600X175-16N, symbol Samacsys:ISO7740FDBQR
- added IC6: ZXTR2105FQ-7, Samacsys:SOT96P240X110-3N, symbol Samacsys:ZXTR2105FQ-7
- added J1, J2, J3: BHR-06-VUA, Samacsys:SHDR6W64P254_2X3_1522X880X920P, symbol Samacsys:BHR-06-VUA
- added J4: 61201021621, Samacsys:SHDR10W64P254_2X5_2036X885X925P, symbol Samacsys:61201021621
- added JPVCC1: VCC, Jumper:SolderJumper-3_P1.3mm_Open_Pad1.0x1.5mm, symbol Jumper:Jumper_3_Open
- added R1, R12: 4.7k, Resistor_SMD:R_1206_3216Metric, symbol Device:R_Small
- renumbered R9 to R10, R10 to R11, R11 to R13, R12 to R14, R13 to R15, R14 to R16, R15 to R17, R16 to R18, R17 to R19, R1 to R2, R18 to R20, R19 to R21, R20 to R22, R21 to R23, R22 to R24, R23 to R25, R24 to R26, R25 to R27, R26 to R28, R27 to R29, R2 to R3, R28 to R30, R3 to R4, R4 to R5, R5 to R6, R6 to R7, R7 to R8, R8 to R9
Connections:
- net +5V: now also C1.2, C2.1, C3.2, C4.2, IC1.9 (COM), IC2.9 (VDD), IC3.1 (VCC1), IC4.1 (VCC1), J1.1, J1.2, J3.1, J3.2, R1.2, R12.2
- net AGND: now also J2.3, J2.4
- net r0: now also IC1.16 (1C)
- net r1: now also IC1.15 (2C)
- net r2: now also IC1.14 (3C)
- net r3: now also IC1.13 (4C)
- net r4: now also IC1.12 (5C)
- net r5: now also IC1.11 (6C)
- net inL: now reaches K1.4, R3.2
- net inL: now also J2.6
- net inR: now reaches K1.5, R2.2
- net inR: now also J2.5
- net outR: now reaches K6.6, R25.1, R29.1
- net outR: now also J2.1
- net outL: now reaches K6.3, R26.1, R30.1
- net outL: now also J2.2
- new net: IC5.10 (7C), J4.10, J4.9
- new net: IC5.16 (1C), J4.3
- new net: IC5.13 (4C), J4.4
- new net: IC5.15 (2C), J4.5
- new net: IC5.12 (5C), J4.6
- new net: IC5.14 (3C), J4.7
- new net: IC5.11 (6C), J4.8
- new net: IC4.14 (OUTA), IC5.1 (1B)
- new net: IC4.13 (OUTB), IC5.2 (2B)
- new net: IC4.12 (OUTC), IC5.3 (3B)
- new net: IC4.11 (OUTD), IC5.4 (4B)
- new net: IC3.13 (OUTB), IC5.5 (5B)
- new net: IC3.12 (OUTC), IC5.6 (6B)
- new net: IC3.11 (OUTD), IC5.7 (7B)
- new net: JPVCC1.3 (B), R1.1
- new net: IC1.1 (1B), IC2.6 (GPB5)
- new net: IC1.2 (2B), IC2.5 (GPB4)
- new net: IC1.3 (3B), IC2.4 (GPB3)
- new net: IC1.4 (4B), IC2.3 (GPB2)
- new net: IC1.5 (5B), IC2.2 (GPB1)
- new net: IC1.6 (6B), IC2.1 (GPB0)
- new net: IC2.21 (GPA0), IC4.3 (INA)
- new net: IC2.22 (GPA1), IC4.4 (INB)
- new net: IC2.23 (GPA2), IC4.5 (INC)
- new net: IC2.24 (GPA3), IC4.6 (IND)
- new net: IC2.18 (~{RESET}), R12.1
- new net: IC2.25 (GPA4), IC3.6 (IND)
- new net: IC2.26 (GPA5), IC3.4 (INB)
- new net: IC2.27 (GPA6), IC3.5 (INC)
- new net +5VI: C5.2, C6.2, C7.1, IC3.10 (EN2), IC3.16 (VCC2), IC4.10 (EN2), IC4.16 (VCC2), IC6.2 (VOUT)
- new net GNDA: C5.1, C6.1, C7.2, C8.1, IC3.15 (GND2_2), IC3.9 (GND2_1), IC4.15 (GND2_2), IC4.9 (GND2_1), IC5.8 (E), IC6.1 (GND), J4.2
- new net GNDD: C1.1, C2.2, C3.1, C4.1, IC1.8 (E), IC2.10 (VSS), IC2.16 (A1), IC2.17 (A2), IC3.2 (GND1_1), IC3.8 (GND1_2), IC4.2 (GND1_1), IC4.8 (GND1_2), J1.3, J1.4, J3.3, J3.4, JPVCC1.1 (A)
- new net SCL: IC2.12 (SCL), J1.5, J3.5
- new net SDA: IC2.13 (SDA), J1.6, J3.6
- new net VCC: C8.2, IC5.9 (COM), IC6.3 (VIN), J4.1
- new net dual: IC2.15 (A0), JPVCC1.2 (C)
- no-connect marks 0 -> 9
Other:
- note removed: "audio output to power amp"
- note removed: "unswitched audio input typically unused"
- moved on the sheet: H1, H2, H3, H4, K1, K2, K3, K4, K5, K6, R10, R11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

Commit message: somehow maybe done
Parts:
- removed C3, C4, C5, C6: .1uf, Capacitor_SMD:C_1206_3216Metric, symbol Device:C_Small
- removed C7: 10uf, Capacitor_SMD:C_1206_3216Metric, symbol Device:C_Small
- removed C8: 1uf, Capacitor_SMD:C_1206_3216Metric, symbol Device:C_Small
- removed IC2: MCP23017T-E_SS, Samacsys:SOP65P780X200-28N, symbol Samacsys:MCP23017T-E_SS
- removed IC3, IC4: ISO7740FDBQR, Samacsys:SOP64P600X175-16N, symbol Samacsys:ISO7740FDBQR
- removed IC5: ULN2003ADR, Samacsys:SOIC127P600X175-16N, symbol Samacsys:ULN2003ADR
- removed IC6: ZXTR2105FQ-7, Samacsys:SOT96P240X110-3N, symbol Samacsys:ZXTR2105FQ-7
- removed J1: BHR-06-VUA, Samacsys:SHDR6W64P254_2X3_1522X880X920P, symbol Samacsys:BHR-06-VUA
- removed J4: 61201021621, Samacsys:SHDR10W64P254_2X5_2036X885X925P, symbol Samacsys:61201021621
- removed JPVCC1: VCC, Jumper:SolderJumper-3_P1.3mm_Open_Pad1.0x1.5mm, symbol Jumper:Jumper_3_Open
- removed R1: 4.7k, Resistor_SMD:R_1206_3216Metric, symbol Device:R_Small
- added J1: PJRAS4X2U01AUX, Samacsys:PJRAS4X2U01AUX, symbol Samacsys:PJRAS4X2U01AUX
- added J3: TFM-105-01-F-D, Samacsys:TFM-105-XX-YYY-D, symbol Samacsys:TFM-105-01-F-D
- added K1, K2, K3, K4: RELAY_G6K, RlxPassiveFootprints:G6K-2F-Y, symbol relaixedPassive-rescue:RELAY_G6K
- renumbered J3 to J4, K6 to K10, K1 to K5, K2 to K6, K3 to K7, K4 to K8, K5 to K9, R2 to R1, R11 to R10, R12 to R11, R13 to R12, R14 to R13, R15 to R14, R16 to R15, R17 to R16, R18 to R17, R19 to R18, R20 to R19, R3 to R2, R21 to R20, R22 to R21, R23 to R22, R24 to R23, R25 to R24, R26 to R25, R27 to R26, R28 to R27, R29 to R28, R30 to R29, R4 to R3, R5 to R4, R6 to R5, R7 to R6, R8 to R7, R9 to R8, R10 to R9
Connections:
- no-connect marks 9 -> 5
